File: minimal-dock/Main.kicad_sch (KiCad schematic)
At the start: 13 parts, among them IC401 TLV70218, X401 Debug, X402 Voltage, X403 Host, X404 Device, X405 UART

Commit message: Replace X404 USB-C plug with Same Sky UP32-C-H-G-SMT-3-P24-TR
The GlobTek PLUG-USBC-241SMT-4BC2SS is out of stock. Add the Same Sky
symbol, footprint and STEP model as project-local libraries, keep all
X404 pin assignments, reroute the connector fanout and set the board
thickness to 1.0 mm.
Parts:
- X404: value Device -> UP32-C-H-G-SMT-3-P24-TR; footprint GlobTect:PLUG-USBC-241SMT-4BC2SS -> SameSky:SAMESKY_UP32-C-H-G-SMT-3-P24-TR; symbol Connector:USB_C_Receptacle -> SameSky:UP32-C-H-G-SMT-3-P24-TR; digikey# 1939-PLUG-USBC-241SMT-4BC2SSCT-ND -> 2223-UP32-C-H-G-SMT-3-P24-TRCT-ND; manf GlobTek, Inc. -> Same Sky; manf# PLUG-USBC-241SMT-4BC2SS -> UP32-C-H-G-SMT-3-P24-TR; mouser# (none) -> 179-UP32CHGSMT3P24TR
Connections:
- net GND: now also X404.SH1 (SHIELD), X404.SH2 (SHIELD); no longer X404.S1 (SHIELD)
